File: PCB_design/_autosave-arduino_dummy_load_pcb.kicad_pcb (KiCad board)
At the start: 2 copper layers, 122 parts, among them J1 Barrel_Jack, J2 Conn_02x08_Odd_Even, U1 MCP3208

Commit message: stuff.
Parts:
- removed the QB1 at (210.8, 87.6)
- moved QB4 135.9 mm to (280.7, 58.4), turned to 270 degrees
- moved RA3 21.9 mm to (103.0, 152.4)
- moved RA6 21.9 mm to (103.0, 154.9)
- moved CB4 12.7 mm to (97.8, 36.8)
Changed lines of the file:
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@@
     (tracks 106)
     (zones 0)
-    (modules 122)
+    (modules 121)
     (nets 60)
   )
@@
   )
   (module Capacitors_SMD:C_0805_HandSoldering (layer F.Cu)
-    (at 85.09 35.56)
+    (at 97.77 36.83)
     (descr "Capacitor SMD 0805, hand soldering")
     (tags "capacitor 0805")
@@
   )
   (module TO_SOT_Packages_THT:TO-220-3_Vertical (layer F.Cu)
-    (at 210.82 87.63)
-    (descr "TO-220-3, Vertical, RM 2.54mm")
-    (tags "TO-220-3 Vertical RM 2.54mm")
-    (fp_text reference QB1 (at 2.54 -3.62) (layer F.SilkS)
-      (effects (font (size 1 1) (thickness 0.15)))
-    )
-    (fp_text value IPP45P03P4L-11 (at 2.54 3.92) (layer F.Fab)
-      (effects (font (size 1 1) (thickness 0.15)))
-    )
-    (fp_text user %R (at 2.54 -3.62) (layer F.Fab)
-      (effects (font (size 1 1) (thickness 0.15)))
-    )
-    (fp_line (start -2.46 -2.5) (end -2.46 1.9) (layer F.Fab) (width 0.1))
-    (fp_line (start -2.46 1.9) (end 7.54 1.9) (layer F.Fab) (width 0.1))
-    (fp_line (start 7.54 1.9) (end 7.54 -2.5) (layer F.Fab) (width 0.1))
-    (fp_line (start 7.54 -2.5) (end -2.46 -2.5) (layer F.Fab) (width 0.1))
-    (fp_line (start -2.46 -1.23) (end 7.54 -1.23) (layer F.Fab) (width 0.1))
-    (fp_line (start 0.69 -2.5) (end 0.69 -1.23) (layer F.Fab) (width 0.1))
-    (fp_line (start 4.39 -2.5) (end 4.39 -1.23) (layer F.Fab) (width 0.1))
-    (fp_line (start -2.58 -2.62) (end 7.66 -2.62) (layer F.SilkS) (width 0.12))
-    (fp_line (start -2.58 2.021) (end 7.66 2.021) (layer F.SilkS) (width 0.12))
-    (fp_line (start -2.58 -2.62) (end -2.58 2.021) (layer F.SilkS) (width 0.12))
-    (fp_line (start 7.66 -2.62) (end 7.66 2.021) (layer F.SilkS) (width 0.12))
-    (fp_line (start -2.58 -1.11) (end 7.66 -1.11) (layer F.SilkS) (width 0.12))
-    (fp_line (start 0.69 -2.62) (end 0.69 -1.11) (layer F.SilkS) (width 0.12))
-    (fp_line (start 4.391 -2.62) (end 4.391 -1.11) (layer F.SilkS) (width 0.12))
-    (fp_line (start -2.71 -2.75) (end -2.71 2.16) (layer F.CrtYd) (width 0.05))
-    (fp_line (start -2.71 2.16) (end 7.79 2.16) (layer F.CrtYd) (width 0.05))
-    (fp_line (start 7.79 2.16) (end 7.79 -2.75) (layer F.CrtYd) (width 0.05))
-    (fp_line (start 7.79 -2.75) (end -2.71 -2.75) (layer F.CrtYd) (width 0.05))
-    (pad 1 thru_hole rect (at 0 0) (size 1.8 1.8) (drill 1) (layers *.Cu *.Mask)
-      (net 27 "Net-(QB1-Pad1)"))
-    (pad 2 thru_hole oval (at 2.54 0) (size 1.8 1.8) (drill 1) (layers *.Cu *.Mask)
-      (net 7 "Net-(CB2-Pad1)"))
-    (pad 3 thru_hole oval (at 5.08 0) (size 1.8 1.8) (drill 1) (layers *.Cu *.Mask)
-      (net 25 "Net-(QB1-Pad3)"))
-    (model ${KISYS3DMOD}/TO_SOT_Packages_THT.3dshapes/TO-220-3_Vertical.wrl
-      (at (xyz 0.1 0 0))
-      (scale (xyz 0.393701 0.393701 0.393701))
-      (rotate (xyz 0 0 0))
-    )
-  )
-  (module TO_SOT_Packages_THT:TO-220-3_Vertical (layer F.Cu)
     (at 274.32 135.89 270)
     (descr "TO-220-3, Vertical, RM 2.54mm")
@@
   )
   (module Resistors_SMD:R_0805_HandSoldering (layer F.Cu)
-    (at 124.54 156.21)
+    (at 102.95 152.4)
     (descr "Resistor SMD 0805, hand soldering")
     (tags "resistor 0805")
@@
   )
   (module Resistors_SMD:R_0805_HandSoldering (layer F.Cu)
-    (at 124.54 158.75)
+    (at 102.95 154.94)
     (descr "Resistor SMD 0805, hand soldering")
     (tags "resistor 0805")
@@
   )
   (module TO_SOT_Packages_THT:TO-220-3_Vertical (layer F.Cu)
-    (at 149.86 21.59)
+    (at 280.67 58.42 270)
     (descr "TO-220-3, Vertical, RM 2.54mm")
     (tags "TO-220-3 Vertical RM 2.54mm")
-    (fp_text reference QB4 (at 2.54 -3.62) (layer F.SilkS)
+    (fp_text reference QB4 (at 2.54 -3.62 270) (layer F.SilkS)
       (effects (font (size 1 1) (thickness 0.15)))
     )
-    (fp_text value IPP45P03P4L-11 (at 2.54 3.92) (layer F.Fab)
+    (fp_text value IPP45P03P4L-11 (at 2.54 -5.08 270) (layer F.Fab)
       (effects (font (size 1 1) (thickness 0.15)))
     )
-    (fp_text user %R (at 2.54 -3.62) (layer F.Fab)
+    (fp_text user %R (at 2.54 -3.62 270) (layer F.Fab)
       (effects (font (size 1 1) (thickness 0.15)))
     )
@@
     (fp_line (start 7.79 2.16) (end 7.79 -2.75) (layer F.CrtYd) (width 0.05))
     (fp_line (start 7.79 -2.75) (end -2.71 -2.75) (layer F.CrtYd) (width 0.05))
-    (pad 1 thru_hole rect (at 0 0) (size 1.8 1.8) (drill 1) (layers *.Cu *.Mask)
+    (pad 1 thru_hole rect (at 0 0 270) (size 1.8 1.8) (drill 1) (layers *.Cu *.Mask)
       (net 2 GND))
-    (pad 2 thru_hole oval (at 2.54 0) (size 1.8 1.8) (drill 1) (layers *.Cu *.Mask)
+    (pad 2 thru_hole oval (at 2.54 0 270) (size 1.8 1.8) (drill 1) (layers *.Cu *.Mask)
       (net 6 BATT_B))
-    (pad 3 thru_hole oval (at 5.08 0) (size 1.8 1.8) (drill 1) (layers *.Cu *.Mask)
+    (pad 3 thru_hole oval (at 5.08 0 270) (size 1.8 1.8) (drill 1) (layers *.Cu *.Mask)
       (net 7 "Net-(CB2-Pad1)"))
     (model ${KISYS3DMOD}/TO_SOT_Packages_THT.3dshapes/TO-220-3_Vertical.wrl
