File: PCB_design/DummyLoad.sch (KiCad schematic (older format))
At the start: 50 parts

Commit message: nearly finished PCB layout and routing
Parts:
- RA10, RA9: footprint Potentiometers:Potentiometer_Trimmer_ACP_CA6v_Horizontal_MountLS -> Potentiometers:Potentiometer_Trimmer_VishaySpectrol_Econtrim-Type36M
