File: PCB_design/arduino_dummy_load_pcb.kicad_pcb (KiCad board)
At the start: 2 copper layers, 209.6 x 109.2 mm, 119 parts, among them J1 Barrel_Jack, J2 Conn_02x08_Odd_Even, J3 Conn_01x01, U1 MCP3208

Commit message: adding to unstable branch
Parts:
- J1: footprint Connectors:JACK_ALIM -> Library:CUI-PJ-002AH-SMT_dc-barrel-jack
- moved J1 6.61 mm to (64.6, 74.9)
Connections:
- J1 pad 1: Net-(J1-Pad1) -> +9V
- J1 pad 2: +9V -> Net-(J1-Pad2)
- J1 pad 3: +9V -> Net-(J1-Pad2)
- REG1 pad 2: Net-(J1-Pad1) -> Net-(J1-Pad2)
Routing:
- net +9V: track 197.8 -> 118.3 mm
- net Net-(J1-Pad1): track 50.3 -> 0.00 mm, vias 1 -> 0
- net Net-(J1-Pad2): track 0.00 -> 22.9 mm
- net (no net): track 0.00 -> 5.78 mm, vias 0 -> 1

Commit message: fixed all of @malcolms problems :)
Routing:
- net +9V: track 118.3 -> 200.6 mm, vias 2 -> 3
- net Net-(J1-Pad2): track 22.9 -> 36.7 mm
- net (no net): track 5.78 -> 0.00 mm, vias 1 -> 0
- net +5V: vias 8 -> 7
Changed lines of the file:
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@@
   (general
     (links 260)
-    (no_connects 5)
-    (area 55.804999 38.024999 265.505001 147.395001)
+    (no_connects 0)
+    (area 43.914287 30.439405 267.970001 149.860001)
     (thickness 1.6)
     (drawings 10)
-    (tracks 609)
+    (tracks 620)
     (zones 0)
     (modules 119)
@@
   (page A4)
   (layers
-    (0 F.Cu signal hide)
+    (0 F.Cu signal)
     (31 B.Cu signal)
     (32 B.Adhes user)
@@
   (gr_line (start 55.88 147.32) (end 265.43 147.32) (layer Edge.Cuts) (width 0.15))
   (gr_line (start 55.88 38.1) (end 55.88 147.32) (layer Edge.Cuts) (width 0.15))
-  (segment (start 71.12 68.529876) (end 71.085378 68.495254) (width 0.508) (layer F.Cu) (net 0))
-  (segment (start 71.12 73.66) (end 71.12 68.529876) (width 0.508) (layer F.Cu) (net 0))
-  (via (at 72.39 68.495254) (size 0.7) (drill 0.4) (layers F.Cu B.Cu) (net 0))
-  (segment (start 66.705888 78.74) (end 67.31 78.74) (width 0.25) (layer B.Cu) (net 0) (status 30))
   (segment (start 78.23794 71.716694) (end 78.23794 72.211668) (width 0.25) (layer F.Cu) (net 1))
-  (segment (start 78.23794 70.82705) (end 78.23794 71.716694) (width 0.25) (layer F.Cu) (net 1))
+  (segment (start 78.23794 70.82705) (end 78.23794 71.716694) (width 0.508) (layer F.Cu) (net 1))
   (segment (start 78.2441 70.82089) (end 78.23794 70.82705) (width 0.25) (layer F.Cu) (net 1))
   (segment (start 78.587939 72.561667) (end 78.23794 72.211668) (width 0.508) (layer B.Cu) (net 1))
@@
   (segment (start 78.2441 68.58) (end 78.2441 70.82089) (width 0.508) (layer F.Cu) (net 1))
   (segment (start 78.2441 64.456282) (end 78.2441 68.58) (width 0.508) (layer F.Cu) (net 1) (status 10))
-  (via (at 78.2441 68.58) (size 0.7) (drill 0.4) (layers F.Cu B.Cu) (net 1))
   (segment (start 99.06 93.03) (end 96.947621 90.917621) (width 0.508) (layer B.Cu) (net 1) (status 10))
   (segment (start 96.947621 90.917621) (end 96.947621 80.437621) (width 0.508) (layer B.Cu) (net 1))
@@
   (segment (start 124.278546 82.029034) (end 124.278546 86.018546) (width 0.25) (layer F.Cu) (net 9) (status 30))
   (segment (start 124.278546 86.018546) (end 124.46 86.2) (width 0.25) (layer F.Cu) (net 9) (status 30))
-  (segment (start 93.98 80.01) (end 104.14 69.85) (width 0.25) (layer F.Cu) (net 10) (status 10))
-  (segment (start 104.14 69.85) (end 119.89 69.85) (width 0.25) (layer F.Cu) (net 10) (status 20))
+  (segment (start 93.98 80.01) (end 104.148528 69.841472) (width 0.25) (layer F.Cu) (net 10))
+  (segment (start 104.148528 69.841472) (end 119.881472 69.841472) (width 0.25) (layer F.Cu) (net 10))
+  (segment (start 119.881472 69.841472) (end 119.89 69.85) (width 0.25) (layer F.Cu) (net 10))
   (segment (start 215.718546 82.029034) (end 215.718546 86.018546) (width 0.25) (layer F.Cu) (net 11) (status 30))
   (segment (start 215.718546 81.579034) (end 210.768546 76.629034) (width 0.25) (layer F.Cu) (net 11) (status 10))
@@
   (segment (start 120.868546 82.029034) (end 120.548546 81.709034) (width 0.25) (layer F.Cu) (net 21) (status 30))
   (segment (start 122.943328 81.897013) (end 123.128205 82.08189) (width 0.25) (layer F.Cu) (net 21) (status 30))
+  (segment (start 150.795849 82.575732) (end 150.795849 130.635385) (width 2.54) (layer B.Cu) (net 22))
+  (segment (start 150.795849 130.635385) (end 150.770117 130.661117) (width 2.54) (layer B.Cu) (net 22))
   (segment (start 150.770117 107.801117) (end 150.770117 100.181117) (width 0.25) (layer B.Cu) (net 22) (status 30))
   (segment (start 138.070117 123.041117) (end 138.070117 115.421117) (width 0.25) (layer B.Cu) (net 22) (status 30))
@@
   (segment (start 137.818275 99.929275) (end 138.070117 100.181117) (width 0.25) (layer F.Cu) (net 22) (status 30))
   (segment (start 147.32 82.55) (end 150.770117 82.55) (width 2.286) (layer B.Cu) (net 22) (status 10))
-  (segment (start 150.770117 82.55) (end 150.770117 130.661117) (width 2.54) (layer B.Cu) (net 22) (status 20))
   (segment (start 138.070117 100.181117) (end 138.070117 130.661117) (width 2.54) (layer B.Cu) (net 22) (status 30))
   (segment (start 238.76 82.55) (end 242.073764 82.55) (width 2.286) (layer B.Cu) (net 23))
@@
   (segment (start 247.636977 58.810833) (end 247.636977 64.27879) (width 0.25) (layer F.Cu) (net 24) (status 20))
   (segment (start 256.86 56.99) (end 249.45781 56.99) (width 0.25) (layer F.Cu) (net 24) (status 10))
+  (segment (start 125.73 70.034759) (end 125.723694 70.041065) (width 0.25) (layer B.Cu) (net 25))
+  (segment (start 125.723694 70.041065) (end 75.121065 70.041065) (width 0.508) (layer B.Cu) (net 25))
+  (segment (start 75.121065 70.041065) (end 74.93 69.85) (width 0.25) (layer B.Cu) (net 25))
+  (segment (start 74.93 69.85) (end 74.31 69.23) (width 0.508) (layer F.Cu) (net 25))
+  (segment (start 74.31 69.23) (end 68.33 69.23) (width 0.508) (layer F.Cu) (net 25))
+  (via (at 74.93 69.85) (size 0.7) (drill 0.4) (layers F.Cu B.Cu) (net 25))
+  (segment (start 125.57647 74.93) (end 125.57647 78.023913) (width 0.508) (layer B.Cu) (net 25))
+  (segment (start 125.57647 70.188289) (end 125.57647 74.93) (width 0.508) (layer B.Cu) (net 25))
+  (segment (start 62.23 69.23) (end 62.03 69.23) (width 1.27) (layer F.Cu) (net 25))
+  (segment (start 62.03 69.23) (end 59.57 71.69) (width 1.27) (layer F.Cu) (net 25))
+  (segment (start 59.57 71.69) (end 59.57 91.772765) (width 1.27) (layer F.Cu) (net 25))
+  (segment (start 59.57 91.772765) (end 59.57 93.03) (width 1.27) (layer F.Cu) (net 25))
+  (segment (start 68.33 69.23) (end 62.23 69.23) (width 1.27) (layer F.Cu) (net 25))
   (segment (start 218.258546 79.947503) (end 216.300768 77.989725) (width 0.508) (layer F.Cu) (net 25))
   (segment (start 126.818546 79.265989) (end 125.57647 78.023913) (width 0.508) (layer F.Cu) (net 25))
   (segment (start 126.818546 82.029034) (end 126.818546 79.265989) (width 0.508) (layer F.Cu) (net 25) (status 10))
-  (segment (start 125.57647 70.188289) (end 125.57647 78.023913) (width 0.508) (layer B.Cu) (net 25))
   (segment (start 125.587631 70.177128) (end 125.57647 70.188289) (width 0.508) (layer B.Cu) (net 25))
   (via (at 125.57647 78.023913) (size 0.7) (drill 0.4) (layers F.Cu B.Cu) (net 25))
@@
   (via (at 216.300768 77.989725) (size 0.7) (drill 0.4) (layers F.Cu B.Cu) (net 25))
   (segment (start 218.258546 82.029034) (end 218.258546 82.479034) (width 0.25) (layer F.Cu) (net 25) (status 30))
-  (segment (start 59.57 86.48) (end 59.57 93.03) (width 1.27) (layer B.Cu) (net 25) (status 20))
   (segment (start 259.410001 61.715903) (end 257.997114 63.12879) (width 0.25) (layer F.Cu) (net 26))
   (segment (start 257.997114 63.12879) (end 257.997114 64.27879) (width 0.25) (layer F.Cu) (net 26) (status 20))
@@
   (segment (start 82.993718 56.6741) (end 83.82 55.847818) (width 0.25) (layer F.Cu) (net 58))
   (segment (start 82.543718 56.6741) (end 82.993718 56.6741) (width 0.25) (layer F.Cu) (net 58) (status 30))
-  (segment (start 75.772319 93.967681) (end 59.57 110.17) (width 1.27) (layer B.Cu) (net 59))
+  (segment (start 62.23 80.63) (end 62.23 107.51) (width 1.27) (layer F.Cu) (net 59))
+  (segment (start 62.23 107.51) (end 59.57 110.17) (width 1.27) (layer F.Cu) (net 59))
+  (segment (start 68.33 80.63) (end 68.13 80.63) (width 1.27) (layer F.Cu) (net 59))
+  (segment (start 68.13 80.63) (end 62.23 80.63) (width 1.27) (layer F.Cu) (net 59))
   (zone (net 2) (net_name GND) (layer B.Cu) (hatch edge 0.508)
     (connect_pads (clearance 0.508))
@@
     (polygon
       (pts
-        (xy 54.61 36.83) (xy 266.7 36.83) (xy 266.7 148.59) (xy 54.61 148.59)
-      )
-    )
-  )
-  (zone (net 1) (net_name +5V) (layer F.Cu) (hatch edge 0.508)
-    (connect_pads (clearance 0.508))
-    (min_thickness 0.254)
-    (fill yes (arc_segments 16) (thermal_gap 0.508) (thermal_bridge_width 0.508))
-    (polygon
-      (pts
-        (xy 165.1 40.64) (xy 165.1 45.72) (xy 99.06 45.72) (xy 99.06 40.64)
+        (xy 266.7 148.59) (xy 54.61 148.59) (xy 54.61 36.83) (xy 266.7 36.83)
       )
     )
